Commit message: ts

File: resources/robots/TOE_dog/urdf/dog.urdf (robot description, URDF)
Before this commit: robot TOE_dog, 18 links, 17 joints
Links:
- link FL_calf: geometry collision box size=0.16 0.0245 0.04; visual mesh filename=../assets/TOE_calf.STL
- link FL_foot: geometry collision sphere radius=0.022; visual mesh filename=../assets/TOE_foot.STL
- link FL_hip: geometry collision cylinder length=0.08 radius=0.046; visual mesh filename=../assets/TOE_FL_hip.STL
- link FL_thigh: geometry collision box size=0.11 0.0245 0.04; visual mesh filename=../assets/TOE_L_thigh.STL
- link FR_calf: geometry collision box size=0.16 0.0245 0.04; visual mesh filename=../assets/TOE_calf.STL
- link FR_foot: geometry collision sphere radius=0.022; visual mesh filename=../assets/TOE_foot.STL
- link FR_hip: geometry collision cylinder length=0.08 radius=0.046; visual mesh filename=../assets/TOE_FR_hip.STL
- link FR_thigh: geometry collision box size=0.11 0.0245 0.04; visual mesh filename=../assets/TOE_R_thigh.STL
- link RL_calf: geometry collision box size=0.16 0.0245 0.04; visual mesh filename=../assets/TOE_calf.STL
- link RL_foot: geometry collision sphere radius=0.022; visual mesh filename=../assets/TOE_foot.STL
- link RL_hip: geometry collision cylinder length=0.08 radius=0.046; visual mesh filename=../assets/TOE_RL_hip.STL
- link RL_thigh: geometry collision box size=0.11 0.0245 0.04; visual mesh filename=../assets/TOE_L_thigh.STL
- link RR_calf: geometry collision box size=0.16 0.0245 0.04; visual mesh filename=../assets/TOE_calf.STL
- link RR_foot: geometry collision sphere radius=0.022; visual mesh filename=../assets/TOE_foot.STL
- link RR_hip: geometry collision cylinder length=0.08 radius=0.046; visual mesh filename=../assets/TOE_RR_hip.STL
- link RR_thigh: geometry collision box size=0.11 0.0245 0.04; visual mesh filename=../assets/TOE_R_thigh.STL
- link base: geometry collision box size=0.27 0.15 0.114; visual mesh filename=../assets/TOE_base.STL
